File: Type.1/dummy_keyboard.kicad_pcb (KiCad board)
At the start: 2 copper layers, 50 x 25 mm, 3 parts, among them SW1 SW_Push

Commit message: update: new goods version.
Parts:
- G***: moved to B.Cu
- moved G*** 6.80 mm to (171.0, 98.5), turned to 180 degrees
Other:
- board text added: "AI/SW과, 정보보안과 그래픽SW과, 경영회계과 빅데이터과, 보건간호과"
- board text added: "Tel. 031-329-4348 https://dukyoung-h.goeyi.kr"
- board text added: "덕영고등학교"
- board text added: "덕영고등학교. DYHS"
- board text removed: "덕영고등학교 소프트웨어부"
