File: Type_7/dummy_keyboard.kicad_pcb (KiCad board)
At the start: 2 copper layers, 50 x 25 mm, 4 parts, among them SW1 SW_Push

Commit message: update: backplate text changed
Other:
- board text added: "경영회계과, 빅데이터과, 보건간호과, 그래픽SW과 인공지능SW과, 정보보안SW과"
- board text removed: "AI/SW과, 정보보안과 그래픽SW과, 경영회계과 빅데이터과, 보건간호과"

Commit message: update: code update
Other:
- board text added: "덕영고등학교 소프트웨어부"
- board text removed: "덕영고등학교. DYHS"
